File: minRead_pcb/E_ink_HAT.kicad_sch (KiCad schematic)
At the start: 28 parts, among them J3 Conn_01x24, Q4 Si1308EDL, Q5 AO3401A, Q6 SS8050

Commit message: - schematic updates: - usb500 mode enabled on bq - charge limit set to 100mA 8.9kohm (safe for small batteries) - series resistors on sd card and epd lines - esd arrays for usb-c and sd-card - increased output cap for ldo from 4.7u to 22u - added pgood to gpio - confirmed reverse polarity stuff - cap to ground instead of series for sd card vdd - fixed cap values on epd
new layout:
- adjusted board size
- very compact
- need to fill ground planes and check drc errors (a lot because of solder mask)
- need to adjust jst footprint in case there's a better choice
- review review review
Parts:
- C18, C19, C20, C21, C22: value 0.1u -> 1u
Connections:
- net RESE: now also Q4.2 (S); no longer Q4.3 (D)
- net at C11.2, D5.1 (K), L1.2: now also Q4.3 (D); no longer Q4.2 (S)
Changed lines of the file:
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@@
 			)
 		)
-		(property "Value" "0.1u"
+		(property "Value" "1u"
 			(at 211.836 90.932 90)
 			(effects
@@
 		(lib_id "Transistor_FET:Si1308EDL")
 		(at 66.04 59.69 0)
-		(unit 1)
-		(exclude_from_sim no)
-		(in_bom yes)
-		(on_board yes)
-		(dnp no)
-		(fields_autoplaced yes)
+		(mirror x)
+		(unit 1)
+		(exclude_from_sim no)
+		(in_bom yes)
+		(on_board yes)
+		(dnp no)
 		(property "Reference" "Q4"
-			(at 72.39 58.4199 0)
+			(at 72.39 60.9601 0)
 			(effects
 				(font
@@
 		)
 		(property "Value" "Si1308EDL"
-			(at 72.39 60.9599 0)
+			(at 72.39 58.4201 0)
 			(effects
 				(font
@@
 		)
 		(property "Footprint" "Package_TO_SOT_SMD:SOT-323_SC-70_Handsoldering"
-			(at 71.12 61.595 0)
+			(at 71.12 57.785 0)
 			(effects
 				(font
@@
 		)
 		(property "Datasheet" "https://www.vishay.com/docs/63399/si1308edl.pdf"
-			(at 71.12 63.5 0)
+			(at 71.12 55.88 0)
 			(effects
 				(font
@@
 			)
 		)
-		(property "Value" "0.1u"
+		(property "Value" "1u"
 			(at 211.836 127.254 90)
 			(effects
@@
 			)
 		)
-		(property "Value" "0.1u"
+		(property "Value" "1u"
 			(at 214.376 119.38 90)
 			(effects
@@
 			)
 		)
-		(property "Value" "0.1u"
+		(property "Value" "1u"
 			(at 211.836 141.986 90)
 			(effects
@@
 			)
 		)
-		(property "Value" "0.1u"
+		(property "Value" "1u"
 			(at 211.836 129.794 90)
 			(effects

Commit message: draft1.0
Parts:
- Q6: footprint Package_TO_SOT_SMD:SOT-23 -> Package_TO_SOT_SMD:SOT-23_Handsoldering
Changed lines of the file:
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@@
 			)
 		)
-		(property "Footprint" "Package_TO_SOT_SMD:SOT-23"
+		(property "Footprint" "Package_TO_SOT_SMD:SOT-23_Handsoldering"
 			(at 177.8 75.946 0)
 			(effects

Commit message: - fixed diode orientation of eink booster - everything works except eink driver: - rst pin pulls high, dc doesn't toggle, etc etc. - TODO for next rev: - remove reset stabilizer and just route 3v3 to epd inductor circuit - replace esd arrays with hand-solderable components (qfn to sot) - replace buttons with resistor ladder circuit (xteink-like) - replace bq24074 with more discrete charging circuit to aid hand-solder - add led driver (15v to 7 series LEDs) - replace usb-c receptacle with through-hole - add external dupont pins for external LED driver access and spare GPIOs
Connections:
- net PREVGH: now also D5.1 (K); no longer D5.2 (A)
- net at C11.2, L1.2, Q4.3 (D): now also D5.2 (A); no longer D5.1 (K)
Other:
- moved on the sheet: D5
Changed lines of the file:
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@@
 	(symbol
 		(lib_id "Diode:MBR0530")
-		(at 68.58 93.98 270)
+		(at 68.58 93.98 90)
 		(unit 1)
 		(exclude_from_sim no)
@@
 		(fields_autoplaced yes)
 		(property "Reference" "D5"
-			(at 71.12 92.3924 90)
+			(at 71.12 93.0274 90)
 			(effects
 				(font
 					(size 1.27 1.27)
 				)
-				(justify left)
+				(justify right)
 			)
 		)
 		(property "Value" "MBR0530"
-			(at 71.12 94.9324 90)
+			(at 71.12 95.5674 90)
 			(effects
 				(font
 					(size 1.27 1.27)
 				)
-				(justify left)
+				(justify right)
 			)
 		)
 		(property "Footprint" "Diode_SMD:D_SOD-123"
-			(at 64.135 93.98 0)
+			(at 73.025 93.98 0)
 			(effects
 				(font

Commit message: gigantic commit, my bad revised schematic to sanity check turns out my fpc was flipped, now fixed added following schematics: - battery protection circuit - series LED driver - external peripheral connector for unused GPIO revised following schematics: - power path, replaced with mcp charger and FET rather than bq - buttons, opted for resistor ladder circuit, added two more for xte compatibility - eink driver, opted to change to updated components from waveshare 2.3 - updated esd components for usb-c and sdmmc - updated usb-c receptacle, now through-hole
New layout:
- mostly same as last time, but work done to ensure good grounding for LED/eink circuits
- eink gpio has minimal crossing/coupling just in case
- esp32 and 24 pin headers have longer pads hopefully for easier soldering
- external header in corner back of device
- prettier passive component layout
- fat 3v3 traces and small zone fill

- todo:
- DRC errors, mostly clearance and silkscreen overlap
Parts:
- removed C10, C11, C13, C14, C15, C16, C17: 4.7u, Capacitor_SMD:C_0805_2012Metric_Pad1.18x1.45mm_HandSolder, symbol Device:C
- removed C12: 0.1u, Capacitor_SMD:C_0805_2012Metric_Pad1.18x1.45mm_HandSolder, symbol Device:C
- removed C18, C19, C20, C21, C22: 1u, Capacitor_SMD:C_0805_2012Metric_Pad1.18x1.45mm_HandSolder, symbol Device:C
- removed D4, D5, D6: MBR0530, Diode_SMD:D_SOD-123, symbol Diode:MBR0530
- removed J3: Conn_01x24, custom:24pin0.5mm, symbol Connector_Generic:Conn_01x24
- removed L1: 68u, Inductor_SMD:L_Changjiang_FNR6028S, symbol Device:L
- removed Q4: Si1308EDL, Package_TO_SOT_SMD:SOT-323_SC-70_Handsoldering, symbol Transistor_FET:Si1308EDL
- removed Q5: AO3401A, Package_TO_SOT_SMD:SOT-23_Handsoldering, symbol Transistor_FET:AO3401A
- removed Q6: SS8050, Package_TO_SOT_SMD:SOT-23_Handsoldering, symbol Transistor_BJT:SS8050
- removed R14: 3, Resistor_SMD:R_0805_2012Metric_Pad1.20x1.40mm_HandSolder, symbol Device:R
- removed R15, R17: 10k, Resistor_SMD:R_0805_2012Metric_Pad1.20x1.40mm_HandSolder, symbol Device:R
- removed R16: 1k, Resistor_SMD:R_0805_2012Metric_Pad1.20x1.40mm_HandSolder, symbol Device:R
- removed R18, R19, R20: 47k, Resistor_SMD:R_0805_2012Metric_Pad1.20x1.40mm_HandSolder, symbol Device:R
Connections:
- no-connect marks 3 -> 0
Other:
- note removed: "Charge Pump"
- note removed: "ESP32 IO"
- note removed: "Reset Stabilizer"
- note removed: "ZIF 24-pin Connector"
