File: minRead_pcb/buttons.kicad_sch (KiCad schematic)
At the start: 6 parts, among them SW1 SW_Push, SW2 SW_Push, SW3 SW_Push, SW4 SW_Push, SW5 SW_Push, SW7 SW_Push

Commit message: - schematic updates: - usb500 mode enabled on bq - charge limit set to 100mA 8.9kohm (safe for small batteries) - series resistors on sd card and epd lines - esd arrays for usb-c and sd-card - increased output cap for ldo from 4.7u to 22u - added pgood to gpio - confirmed reverse polarity stuff - cap to ground instead of series for sd card vdd - fixed cap values on epd
new layout:
- adjusted board size
- very compact
- need to fill ground planes and check drc errors (a lot because of solder mask)
- need to adjust jst footprint in case there's a better choice
- review review review
Parts:
- SW1, SW4, SW5, SW7: footprint Button_Switch_SMD:SW_SPST_TS-1088-xR025 -> Button_Switch_THT:SW_Tactile_SPST_Angled_PTS645Vx39-2LFS
- SW2, SW3: footprint Button_Switch_SMD:SW_SPST_TS-1088-xR025 -> Button_Switch_SMD:SW_SPST_PTS810
Changed lines of the file:
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@@
 			)
 		)
-		(property "Footprint" "Button_Switch_SMD:SW_SPST_TS-1088-xR025"
+		(property "Footprint" "Button_Switch_SMD:SW_SPST_PTS810"
 			(at 152.4 83.82 0)
 			(effects
@@
 			)
 		)
-		(property "Footprint" "Button_Switch_SMD:SW_SPST_TS-1088-xR025"
+		(property "Footprint" "Button_Switch_SMD:SW_SPST_PTS810"
 			(at 125.73 83.82 0)
 			(effects
@@
 			)
 		)
-		(property "Footprint" "Button_Switch_SMD:SW_SPST_TS-1088-xR025"
+		(property "Footprint" "Button_Switch_THT:SW_Tactile_SPST_Angled_PTS645Vx39-2LFS"
 			(at 139.7 132.08 0)
 			(effects
@@
 			)
 		)
-		(property "Footprint" "Button_Switch_SMD:SW_SPST_TS-1088-xR025"
+		(property "Footprint" "Button_Switch_THT:SW_Tactile_SPST_Angled_PTS645Vx39-2LFS"
 			(at 139.7 71.12 0)
 			(effects
@@
 			)
 		)
-		(property "Footprint" "Button_Switch_SMD:SW_SPST_TS-1088-xR025"
+		(property "Footprint" "Button_Switch_THT:SW_Tactile_SPST_Angled_PTS645Vx39-2LFS"
 			(at 139.7 118.11 0)
 			(effects
@@
 			)
 		)
-		(property "Footprint" "Button_Switch_SMD:SW_SPST_TS-1088-xR025"
+		(property "Footprint" "Button_Switch_THT:SW_Tactile_SPST_Angled_PTS645Vx39-2LFS"
 			(at 139.7 96.52 0)
 			(effects

Commit message: gigantic commit, my bad revised schematic to sanity check turns out my fpc was flipped, now fixed added following schematics: - battery protection circuit - series LED driver - external peripheral connector for unused GPIO revised following schematics: - power path, replaced with mcp charger and FET rather than bq - buttons, opted for resistor ladder circuit, added two more for xte compatibility - eink driver, opted to change to updated components from waveshare 2.3 - updated esd components for usb-c and sdmmc - updated usb-c receptacle, now through-hole
New layout:
- mostly same as last time, but work done to ensure good grounding for LED/eink circuits
- eink gpio has minimal crossing/coupling just in case
- esp32 and 24 pin headers have longer pads hopefully for easier soldering
- external header in corner back of device
- prettier passive component layout
- fat 3v3 traces and small zone fill

- todo:
- DRC errors, mostly clearance and silkscreen overlap
Parts:
- removed SW1, SW4, SW5, SW7: SW_Push, Button_Switch_THT:SW_Tactile_SPST_Angled_PTS645Vx39-2LFS, symbol Switch:SW_Push
- removed SW2, SW3: SW_Push, Button_Switch_SMD:SW_SPST_PTS810, symbol Switch:SW_Push
